Commit message: idk

File: description/camera.xacro (robot description, xacro)
@@ -4,5 +4,5 @@
         <parent link="chassis"/>
         <child link="camera_link"/>
-        <origin xyz="0.305 0 0.08" rpy="0 0 0"/>
+        <origin xyz="0.276 0 0.181" rpy="0 0.18 0"/>
     </joint>
     <link name="camera_link">

File: description/robot.urdf.xacro (robot description, xacro)
@@ -1,8 +1,14 @@
 <?xml version="1.0"?>
 <robot xmlns:xacro="http://www.ros.org/wiki/xacro"  name="robot">
+    <xacro:arg name="use_ros2_control" default="true"/>
     <xacro:include filename="robot_core.xacro" />
-   <!-- <xacro:include filename="gazebo_control.xacro" /> -->
-   <xacro:include filename="ros2_control.xacro">
+    <xacro:if value="$(arg use_ros2_control)">
+        <xacro:include filename="ros2_control.xacro" />
+    </xacro:if>
+    <xacro:unless value="$(arg use_ros2_control)">
+        <xacro:include filename="gazebo_control.xacro" />
+    </xacro:unless>
     <xacro:include filename="lidar.xacro" />
     <xacro:include filename="camera.xacro" />
+    <!-- <xacro:include filename="depth_camera.xacro" /> -->
 </robot>

File: description/robot_core.xacro (robot description, xacro)
@@ -19,4 +19,12 @@
 <!-- Base link-->
 <link name="base_link">
+</link>
+<!-- BASE_FOOTPRINT LINK -->
+<joint name="base_footprint_joint" type="fixed">
+    <parent link="base_link"/>
+    <child link="base_footprint"/>
+    <origin xyz="0 0 0" rpy="0 0 0"/>
+</joint>
+<link name="base_footprint">
 </link>
 <!-- chassis link-->
@@ -63,5 +71,5 @@
     <collision>
         <geometry>
-            <cylinder length="0.04" radius="0.05" />
+            <sphere length="0.04" radius="0.05" />
         </geometry>
     </collision>
@@ -89,5 +97,5 @@
     <collision>
         <geometry>
-            <cylinder length="0.04" radius="0.05" />
+            <sphere length="0.04" radius="0.05" />
         </geometry>
     </collision>
